File: IoThermometer.sch (KiCad schematic (older format))
At the start: 7 parts, among them U1 NodeMCU_Amica_R2, U2 DS18B20

Commit message: adjusted pcb size
Parts:
- D1, D2: footprint LEDs:LED_0805 -> LED_THT:LED_D5.0mm; symbol LED -> Device:LED
- R1, R2, R3: footprint Resistors_SMD:R_0805_HandSoldering -> Resistor_THT:R_Axial_DIN0207_L6.3mm_D2.5mm_P7.62mm_Horizontal; symbol R -> Device:R
- U1: symbol NodeMCU_Amica_R2 -> nodemcu:NodeMCU_Amica_R2
- U2: footprint Housings_SOIC:SOIC-8-1EP_3.9x4.9mm_Pitch1.27mm -> Sensors:DHT22_Temperature_Humidity; symbol DS18B20 -> IoThermometer-rescue:DS18B20
Connections:
- wire segments 29 -> 34
Other:
- note added: "D3, D4, D8 output only - used to determine boot mode"
- moved on the sheet: U2

Commit message: change dht22 symbol, fix pinout in footprint
Parts:
- removed U2: DS18B20, Sensors:DHT22_Temperature_Humidity, symbol IoThermometer-rescue:DS18B20
- added TH1: DHT22_Temperature_Humidity, Sensors:DHT22_Temperature_Humidity, symbol sensors:DHT22_Temperature_Humidity
Changed lines of the file:
@@
 L power:GND #PWR03
 U 1 1 589EA34C
-P 4400 3550
-F 0 "#PWR03" H 4400 3300 50  0001 C CNN
-F 1 "GND" H 4400 3400 50  0000 C CNN
-F 2 "" H 4400 3550 50  0000 C CNN
-F 3 "" H 4400 3550 50  0000 C CNN
-	1    4400 3550
+P 4500 3550
+F 0 "#PWR03" H 4500 3300 50  0001 C CNN
+F 1 "GND" H 4500 3400 50  0000 C CNN
+F 2 "" H 4500 3550 50  0000 C CNN
+F 3 "" H 4500 3550 50  0000 C CNN
+	1    4500 3550
 	0    -1   -1   0
 $EndComp
@@
 L Device:LED D2
 U 1 1 589EA47E
-P 4700 5500
-F 0 "D2" H 4700 5600 50  0000 C CNN
-F 1 "LED" H 4700 5400 50  0000 C CNN
-F 2 "LED_THT:LED_D5.0mm" H 4700 5500 50  0001 C CNN
-F 3 "" H 4700 5500 50  0000 C CNN
-F 4 "LY R976-PS-36" H 4700 5500 60  0001 C CNN "MPN"
-F 5 "http://www.digikey.com/short/32pnmb" H 4700 5500 60  0001 C CNN "URL"
-F 6 "amber" H 4700 5500 60  0001 C CNN "Color"
-	1    4700 5500
+P 4700 4700
+F 0 "D2" H 4700 4800 50  0000 C CNN
+F 1 "LED" H 4700 4600 50  0000 C CNN
+F 2 "LED_THT:LED_D5.0mm" H 4700 4700 50  0001 C CNN
+F 3 "" H 4700 4700 50  0000 C CNN
+F 4 "LY R976-PS-36" H 4700 4700 60  0001 C CNN "MPN"
+F 5 "http://www.digikey.com/short/32pnmb" H 4700 4700 60  0001 C CNN "URL"
+F 6 "amber" H 4700 4700 60  0001 C CNN "Color"
+	1    4700 4700
 	0    -1   -1   0
 $EndComp
@@
 L Device:R R2
 U 1 1 589EA7A6
-P 4700 5050
-F 0 "R2" V 4780 5050 50  0000 C CNN
-F 1 "330" V 4700 5050 50  0000 C CNN
-F 2 "Resistor_THT:R_Axial_DIN0207_L6.3mm_D2.5mm_P7.62mm_Horizontal" V 4630 5050 50  0001 C CNN
-F 3 "" H 4700 5050 50  0000 C CNN
-F 4 "RC0805JR-07330RL" V 4700 5050 60  0001 C CNN "MPN"
-F 5 "http://www.digikey.com/short/32pnmn" V 4700 5050 60  0001 C CNN "URL"
-F 6 "0.125W" V 4700 5050 60  0001 C CNN "Power_Rating"
-	1    4700 5050
+P 4700 4250
+F 0 "R2" V 4780 4250 50  0000 C CNN
+F 1 "330" V 4700 4250 50  0000 C CNN
+F 2 "Resistor_THT:R_Axial_DIN0207_L6.3mm_D2.5mm_P7.62mm_Horizontal" V 4630 4250 50  0001 C CNN
+F 3 "" H 4700 4250 50  0000 C CNN
+F 4 "RC0805JR-07330RL" V 4700 4250 60  0001 C CNN "MPN"
+F 5 "http://www.digikey.com/short/32pnmn" V 4700 4250 60  0001 C CNN "URL"
+F 6 "0.125W" V 4700 4250 60  0001 C CNN "Power_Rating"
+	1    4700 4250
 	-1   0    0    1
 $EndComp
@@
 L power:GND #PWR07
 U 1 1 589EA897
-P 4700 5850
-F 0 "#PWR07" H 4700 5600 50  0001 C CNN
-F 1 "GND" H 4700 5700 50  0000 C CNN
-F 2 "" H 4700 5850 50  0000 C CNN
-F 3 "" H 4700 5850 50  0000 C CNN
-	1    4700 5850
+P 4700 5050
+F 0 "#PWR07" H 4700 4800 50  0001 C CNN
+F 1 "GND" H 4700 4900 50  0000 C CNN
+F 2 "" H 4700 5050 50  0000 C CNN
+F 3 "" H 4700 5050 50  0000 C CNN
+	1    4700 5050
 	1    0    0    -1
 $EndComp
@@
 	3650 3550 3700 3550
 Wire Wire Line
-	4250 3550 4400 3550
+	4350 3550 4500 3550
 Wire Wire Line
 	7750 2500 7750 2750
@@
 	5200 2350 5200 2600
 Connection ~ 5200 2600
-$Comp
-L IoThermometer-rescue:DS18B20 U2
-U 1 1 58BAF9C6
-P 4150 3250
-F 0 "U2" H 4000 3500 50  0000 C CNN
-F 1 "DS18B20" H 4150 3000 50  0000 C CNN
-F 2 "Sensors:DHT22_Temperature_Humidity" H 4000 3500 50  0001 C CNN
-F 3 "" H 4000 3500 50  0000 C CNN
-F 4 "DS18B20Z+" H 4150 3250 60  0001 C CNN "MPN"
-F 5 "http://www.digikey.com/short/32pnmp" H 4150 3250 60  0001 C CNN "URL"
-	1    4150 3250
-	0    -1   -1   0
-$EndComp
 $Comp
 L Device:R R3
@@
 	5250 3900 4700 3900
 Wire Wire Line
-	4700 3900 4700 4900
-Wire Wire Line
-	4700 5200 4700 5350
-Wire Wire Line
-	4700 5650 4700 5850
+	4700 3900 4700 4100
+Wire Wire Line
+	4700 4400 4700 4550
+Wire Wire Line
+	4700 4850 4700 5050
 Wire Wire Line
 	4150 3800 5250 3800
+$Comp
+L sensors:DHT22_Temperature_Humidity TH1
+U 1 1 5E2D39A3
+P 4200 3550
+F 0 "TH1" H 3750 4100 60  0000 L CNN
+F 1 "DHT22_Temperature_Humidity" H 2600 3800 60  0000 L CNN
+F 2 "Sensors:DHT22_Temperature_Humidity" H 4200 3550 60  0001 C CNN
+F 3 "" H 4200 3550 60  0000 C CNN
+	1    4200 3550
+	1    0    0    -1
+$EndComp
 $EndSCHEMATC

Commit message: resize resistors & change about text
Parts:
- R1, R2, R3: footprint Resistor_THT:R_Axial_DIN0207_L6.3mm_D2.5mm_P7.62mm_Horizontal -> Resistor_THT:R_Axial_DIN0207_L6.3mm_D2.5mm_P10.16mm_Horizontal
Changed lines of the file:
@@
 F 0 "R1" V 7830 2900 50  0000 C CNN
 F 1 "330" V 7750 2900 50  0000 C CNN
-F 2 "Resistor_THT:R_Axial_DIN0207_L6.3mm_D2.5mm_P7.62mm_Horizontal" V 7680 2900 50  0001 C CNN
+F 2 "Resistor_THT:R_Axial_DIN0207_L6.3mm_D2.5mm_P10.16mm_Horizontal" V 7680 2900 50  0001 C CNN
 F 3 "" H 7750 2900 50  0000 C CNN
 F 4 "RC0805JR-07330RL" V 7750 2900 60  0001 C CNN "MPN"
@@
 F 0 "R2" V 4780 4250 50  0000 C CNN
 F 1 "330" V 4700 4250 50  0000 C CNN
-F 2 "Resistor_THT:R_Axial_DIN0207_L6.3mm_D2.5mm_P7.62mm_Horizontal" V 4630 4250 50  0001 C CNN
+F 2 "Resistor_THT:R_Axial_DIN0207_L6.3mm_D2.5mm_P10.16mm_Horizontal" V 4630 4250 50  0001 C CNN
 F 3 "" H 4700 4250 50  0000 C CNN
 F 4 "RC0805JR-07330RL" V 4700 4250 60  0001 C CNN "MPN"
@@
 F 0 "R3" V 3980 3800 50  0000 C CNN
 F 1 "4.7k" V 3900 3800 50  0000 C CNN
-F 2 "Resistor_THT:R_Axial_DIN0207_L6.3mm_D2.5mm_P7.62mm_Horizontal" V 3830 3800 50  0001 C CNN
+F 2 "Resistor_THT:R_Axial_DIN0207_L6.3mm_D2.5mm_P10.16mm_Horizontal" V 3830 3800 50  0001 C CNN
 F 3 "" H 3900 3800 50  0000 C CNN
 F 4 "RC0805FR-074K7L" V 3900 3800 60  0001 C CNN "MPN"
